File: kicad/stm32h743_core.kicad_sch (KiCad schematic)
At the start: 77 parts, among them J1 GPIO, J2 GPIO, J3 USB_C, J4 SWD, J5 BOOT, J6 5VIN, SW1 NRST_KEY, SW2 USER_KEY, U1 STM32H743ZIT6, U2 TPS54331DDAR, U3 USBLC6-2SC6, X1 8MHz, X2 32.768kHz

Commit message: feat: 执行层策略——SS 电容 C28、DSN 层类约束、飞线预布线改 B.Cu
- 规格/生成器: TPS54331 SS 外接 C28 10nF(TI §7.3.5 内部无软启动)
- 网表门禁: VCAP 单网、3V3_SW 迁移、SS 规则、LED 极性同步
- gen_pcb: 飞线预布线全部改 B.Cu(层策略), 过孔入盘 0.4/0.2, R14 挪位+C48
- pipeline: DSN 按层策略分四类(GND/P3V3/POW5/Default)带 use_layer 约束
- 状态: 层策略门禁首次通过; DRC 25 未连通+7 error, 收敛方案待决策
Parts:
- added C28: 10n, Capacitor_SMD:C_0402_1005Metric, symbol Device:C
Connections:
- net +3V3: now also C28.2
- net SS: now reaches U2.4 (SS)
- net SS: now also C28.1
